Commit message: viz: build depends and launch fixes

File: z_laser_viz/urdf/zlp1.urdf.xacro (robot description, xacro)
@@ -6,5 +6,5 @@
             <origin xyz="0.245 0.04 0" rpy="${pi} ${pi/2} 0"/>
             <geometry>
-                <mesh filename="file://$(find z_laser_simulator)/meshes/zlp1.dae"/>
+                <mesh filename="file://$(find z_laser_viz)/meshes/zlp1.dae"/>
             </geometry>
         </visual>
@@ -12,5 +12,5 @@
             <origin xyz="0.245 0.04 0" rpy="${pi} ${pi/2} 0"/>
             <geometry>
-                <mesh filename="file://$(find z_laser_simulator)/meshes/zlp1.stl"/>
+                <mesh filename="file://$(find z_laser_viz)/meshes/zlp1.stl"/>
             </geometry>
         </collision>
